File: 01 Raspberry Hat 5 Schematic.sch (EAGLE design)
At the start: 86 parts, among them IC1 L298, IC2 L298, Q2 8 MHz, T14 BSS306N, U1 STM32F051C8T, U2 SN74LVC4245APWR, U3 SN74LVC4245APWR

Commit message: Upload version 5.0.0
Parts:
- removed LED, MOT1, MOT2, MOT3, MOT4, POWER_CON: (no value), con-ptr500:AK500/2
- removed SERVO: C-GRID-06-70543, con-molex:C-GRID-06-70543
- added X4: 2510-, con-3m:2510-
- added X6: 1751303, con-phoenix-350:1751303
- added X7: 1751248, con-phoenix-350:1751248
- X2: value (none) -> 2508-; device con-phoenix-254:MPT2 -> Simplex-Connectors:2508-
- X3: value (none) -> MC2; device con-phoenix-254:MPT2 -> con-phoenix-381_l:MC2
Connections:
- new net DATA+: X2-4.KL
- new net DATA-: X2-3.KL
- new net SCL_TX: U1PB.PB10, X4-5.KL
- new net SDA_RX: U1PB.PB11, X4-3.KL, X4-4.KL
- net +5V: now also X2-2.KL
- net +7V/1: no longer SERVO-1.S, X2-2.1
- net +7V/2: no longer SERVO-2.S, X2-1.1
- net GND: now also X2-8.KL, X3.1.SK, X4-10.KL, X4-9.KL; no longer POWER_CON-1.KL, SERVO-6.S, X3-2.1
- net IN21_UC: now also U1PA.PA11; no longer U1PB.PB10
- net IN22_UC: now also U1PA.PA12; no longer U1PB.PB11
- net MOT11: now also X6-7.K; no longer MOT1-1.KL
- net MOT12: now also X6-8.K; no longer MOT1-2.KL
- net MOT21: now also X6-5.K; no longer MOT2-1.KL
- net MOT22: now also X6-6.K; no longer MOT2-2.KL
- net MOT31: now also X6-3.K; no longer MOT3-1.KL
- net MOT32: now also X6-4.K; no longer MOT3-2.KL
- net MOT41: now also X6-1.K; no longer MOT4-1.KL
- net MOT42: now also X6-2.K; no longer MOT4-2.KL
- net N$24: now also X7-1.K; no longer LED-1.KL
- net RPI_CLK: now also X2-7.KL
- net RPI_MISO: now also X2-5.KL
- net RPI_MOSI: now also X2-6.KL
- net SERVO1: now also X4-6.KL; no longer SERVO-3.S
- net SERVO2: now also X4-7.KL; no longer SERVO-4.S
- net SERVO3: now also X4-8.KL; no longer SERVO-5.S
- net VCC: now also X2-1.KL, X3.2.SK, X7-2.K; no longer LED-2.KL, POWER_CON-2.KL, X3-1.1
Other:
- note added: "Manipulator + USB"
- note removed: "Manipulator control"
- note removed: "may be connected if only 1 PS is enough"
