File: 01 Raspberry Hat 6 Schematic.brd (EAGLE design)
At the start: 100 x 68 mm, 83 parts, among them IC1 L298, IC2 L298, Q2 8 MHz, T14 BSS306N, U1 STM32F051C8T, U2 SN74LVC4245APWR, U3 SN74LVC4245APWR, X2 2508-, X3 MC2, X4 2510-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

Commit message: Upload version 6.0.0
Connections:
- net GND: now also X2.1
- net VCC: no longer X2.1
Routing:
- net VCC: track 264.2 -> 250.9 mm
- net +5V: track 308.1 -> 306.2 mm
- net GND: vias 34 -> 37
