File: 01 Raspberry Hat 6 Schematic.sch (EAGLE design)
At the start: 82 parts, among them IC1 L298, IC2 L298, Q2 8 MHz, T14 BSS306N, U1 STM32F051C8T, U2 SN74LVC4245APWR, U3 SN74LVC4245APWR, X2 2508-, X3 MC2, X4 2510-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

Commit message: Upload version 6.0.0
Parts:
- added X5: (no value), con-phoenix-254:MPT2
- R46: value 2k2 -> 1k
Connections:
- net +5V: now also X4-3.KL
- net +7V/1: now also X4-1.KL
- net +7V/2: now also X4-2.KL
- net DATA+: now also X5-2.1
- net DATA-: now also X5-1.1
- net SDA_RX: no longer X4-3.KL
Changed lines of the file:
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@@
 <?xml version="1.0" encoding="utf-8"?>
 <!DOCTYPE eagle SYSTEM "eagle.dtd">
-<eagle version="7.7.0">
+<eagle version="8.5.2">
 <drawing>
 <settings>
 <setting alwaysvectorfont="no"/>
+<setting keepoldvectorfont="yes"/>
 <setting verticaltext="up"/>
 </settings>
@@
 <part name="SUPPLY7" library="supply2" deviceset="VCC" device=""/>
 <part name="R45" library="resistor" deviceset="R-EU_" device="M0805" value="10k"/>
-<part name="R46" library="resistor" deviceset="R-EU_" device="M0805" value="2k2"/>
+<part name="R46" library="resistor" deviceset="R-EU_" device="M0805" value="1k"/>
 <part name="GND42" library="supply1" deviceset="GND" device=""/>
 <part name="C20" library="resistor" deviceset="C-EU" device="C0805" value="47u">
@@
 <part name="X3" library="con-phoenix-381_l" deviceset="MC2" device=""/>
 <part name="X2" library="Simplex-Connectors" deviceset="2508-" device=""/>
+<part name="SUPPLY12" library="supply2" deviceset="+7V" device="" value="+7V/1"/>
+<part name="SUPPLY13" library="supply2" deviceset="+7V" device="" value="+7V/2"/>
+<part name="X5" library="con-phoenix-254" deviceset="MPT2" device=""/>
 </parts>
 <sheets>
@@
 <instance part="X2" gate="-7" x="246.38" y="63.5"/>
 <instance part="X2" gate="-8" x="246.38" y="60.96"/>
+<instance part="SUPPLY12" gate="G$1" x="256.54" y="121.92"/>
+<instance part="SUPPLY13" gate="G$1" x="264.16" y="121.92"/>
+<instance part="X5" gate="-1" x="276.86" y="55.88"/>
+<instance part="X5" gate="-2" x="276.86" y="50.8"/>
 </instances>
 <busses>
@@
 <pinref part="X2" gate="-2" pin="KL"/>
 </segment>
+<segment>
+<pinref part="X4" gate="-3" pin="KL"/>
+<wire x1="251.46" y1="111.76" x2="269.24" y2="111.76" width="0.1524" layer="91"/>
+<wire x1="269.24" y1="111.76" x2="269.24" y2="119.38" width="0.1524" layer="91"/>
+<pinref part="P+5" gate="1" pin="+5V"/>
+</segment>
 </net>
 <net name="RPI_CLK" class="0">
@@
 <junction x="307.34" y="157.48"/>
 </segment>
+<segment>
+<pinref part="X4" gate="-1" pin="KL"/>
+<pinref part="SUPPLY12" gate="G$1" pin="+7V"/>
+<wire x1="251.46" y1="116.84" x2="256.54" y2="116.84" width="0.1524" layer="91"/>
+<wire x1="256.54" y1="116.84" x2="256.54" y2="119.38" width="0.1524" layer="91"/>
+</segment>
 </net>
 <net name="+7V/2" class="0">
@@
 <pinref part="C10" gate="G$1" pin="1"/>
 <junction x="340.36" y="157.48"/>
+</segment>
+<segment>
+<pinref part="X4" gate="-2" pin="KL"/>
+<pinref part="SUPPLY13" gate="G$1" pin="+7V"/>
+<wire x1="251.46" y1="114.3" x2="264.16" y2="114.3" width="0.1524" layer="91"/>
+<wire x1="264.16" y1="114.3" x2="264.16" y2="119.38" width="0.1524" layer="91"/>
 </segment>
 </net>
@@
 </segment>
 <segment>
-<pinref part="X4" gate="-3" pin="KL"/>
-<wire x1="251.46" y1="111.76" x2="269.24" y2="111.76" width="0.1524" layer="91"/>
-<wire x1="269.24" y1="111.76" x2="269.24" y2="119.38" width="0.1524" layer="91"/>
-<pinref part="P+5" gate="1" pin="+5V"/>
-</segment>
-<segment>
 <pinref part="X4" gate="-4" pin="KL"/>
 <wire x1="251.46" y1="109.22" x2="254" y2="109.22" width="0.1524" layer="91"/>
@@
 <pinref part="X2" gate="-3" pin="KL"/>
 </segment>
+<segment>
+<pinref part="X5" gate="-1" pin="1"/>
+<wire x1="274.32" y1="55.88" x2="271.78" y2="55.88" width="0.1524" layer="91"/>
+<label x="271.78" y="55.88" size="0.8128" layer="95" rot="R180" xref="yes"/>
+</segment>
 </net>
 <net name="DATA+" class="0">
@@
 <pinref part="X2" gate="-4" pin="KL"/>
 </segment>
-</net>
+<segment>
+<pinref part="X5" gate="-2" pin="1"/>
+<wire x1="274.32" y1="50.8" x2="271.78" y2="50.8" width="0.1524" layer="91"/>
+<label x="271.78" y="50.8" size="0.8128" layer="95" rot="R180" xref="yes"/>
+</segment>
+</net>
