File: electronics-shield.sch (EAGLE design)
At the start: 76 parts, among them IC1 LINEAR_MCP1703CB, J2 MICRO_USB, Q1 8 MHz, Q2 USER-SUBMITTED_MOSFET-PCHANNE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, Q3 ON-SEMICONDUCTOR---NTZD3154NT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, Q4 ON-SEMICONDUCTOR---NTZD3154NT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, U1 TLE9201SG, U2 TLE9201SG, U3 TLE9201SG, U4 TLE9201SG, U5 STM32F0XX8T, U8 EEPROM-I2C

Commit message: Thermal vias and led for checking voltages added
Parts:
- removed J2: MICRO_USB, electronics-shield:MICRO_USB
- removed JP10: gniazdo IDC męskie 6pin proste, Kell Ideas:ML6
- removed JP4: Listwa kołkowa 2.54mm prosta 1x3 (3pin), Kell Ideas:PINHD-1X3_DNP
- removed JP5: Listwa stykowa 2.54mm prosta 2x20 (40-pin), wydłużona, Kell Ideas:RASPBERRY_PI_B+_TPLACE
- removed Q4: ON-SEMICONDUCTOR---NTZD3154NT1G_ON_SEMICONDUCTOR_NTZD3154NT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, electronics-shield:ON-SEMICONDUCTOR---NTZD3154NT1G_ON_SEMICONDUCTOR_NTZD3154NT1GON_SEMICONDUCTOR_NTZD3154NT1G_0_0
- removed U5: STM32F0XX8T, Kell Ideas:STM32F0XX8T
- removed U8: EEPROM-I2C, Kell Ideas:EEPROM-I2C
- added $3_0_$_2018-08-14_21-12-08: Moduł przetwornicy DC-DC Step-down 4.5..28V --- regulowane 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, Kell Ideas:MP1584_MODULE
- added IC2: TLE9201SG, Kell Ideas:TLE9201SG
- added IC5: LINEAR_MCP1703CB, electronics-shield:LINEAR_MCP1703CB
- added J1: USB-MICRO-B, Kell Ideas:USB-MICRO-B
- added JP1: Listwa kołkowa 2.54mm prosta 1x3 (3pin), Kell Ideas:PINHD-1X3_DNP
- added LED1, LED2, LED3, LED4, LED5: LEDCHIPLED_0603, audio amplifier example:LEDCHIPLED_0603
- added R1, R4: 10k, Kell Ideas:RESISTOR_SMD
- added R13: 200, Kell Ideas:RESISTOR_SMD
- added R2, R3: 4k7, Kell Ideas:RESISTOR_SMD
- added SV2: (no value), Kell Ideas:ML10
- added Y1: 8 MHz, Kell Ideas:CRYSTAL
- IC1: value LINEAR_MCP1703CB -> TLE9201SG; device electronics-shield:LINEAR_MCP1703CB -> Kell Ideas:TLE9201SG
- PCB1: value Moduł przetwornicy DC-DC Step-down 4.5..28V --- regulowane 0.8..20V MP1584 -> Listwa stykowa 2.54mm prosta 2x20 (40-pin), wydłużona; device Kell Ideas:MP1584_MODULE -> Kell Ideas:RASPBERRY_PI_B+_TPLACE
- Q1: value 8 MHz -> USER-SUBMITTED_MOSFET-PCHANNELSMD; device Kell Ideas:CRYSTAL -> electronics-shield:USER-SUBMITTED_MOSFET-PCHANNELSMD; LINK YIC 49SLMT 8.00MHZ 20PF 30PPM -> (none)
- Q2: value USER-SUBMITTED_MOSFET-PCHANNELSMD -> ON-SEMICONDUCTOR---NTZD3154NT1G_ON_SEMICONDUCTOR_NTZD3154NT1GON_SEMICONDUCTOR_NTZD3154NT1G_0_0; device electronics-shield:USER-SUBMITTED_MOSFET-PCHANNELSMD -> electronics-shield:ON-SEMICONDUCTOR---NTZD3154NT1G_ON_SEMICONDUCTOR_NTZD3154NT1GON_SEMICONDUCTOR_NTZD3154NT1G_0_0
- R10: value 100k -> 330
- R11: value 10k -> 330
- R12: value 1k -> 200
- R6: value 4k7 -> 100k
- R7: value 4k7 -> 10k
- R8: value 10k -> 1k
- R9: value 10k -> 1.5k
- SV1: value (none) -> gniazdo IDC męskie 6pin proste; device Kell Ideas:ML10 -> Kell Ideas:ML6
- U1: value TLE9201SG -> STM32F0XX8T; device Kell Ideas:TLE9201SG -> Kell Ideas:STM32F0XX8T
- U2: value TLE9201SG -> EEPROM-I2C; device Kell Ideas:TLE9201SG -> Kell Ideas:EEPROM-I2C
- renumbered C23 to C19, C24 to C20, JP9 to X2, PCB2 to $3_1_$_2018-08-14_21-12-08, PCB3 to $3_2_$_2018-08-14_21-12-08, U$1 to SV3, U$2 to X1, U$5 to SJ1, U$6 to SJ2, U3 to IC3, U4 to IC4
Connections:
- new net N$1: LED1.C, R9.1
- new net N$2: LED2.C, R10.1
- new net N$3: LED3.C, R11.1
- new net N$4: LED4.C, R12.1
- new net N$5: LED5.C, R13.1
- net +3V3: now also IC1.VSO, IC2.VSO, LED5.A, Q2A.G1, Q2B.G2, R1.2, R2.2, R3.2, R4.2, SV1.4, U1PWR.VDD, U1PWR.VDDA, U2.VCC, U2.WP; no longer JP10.4, Q4A.G1, Q4B.G2, R5.2, R6.2, R7.2, R8.2, U1.VSO, U2.VSO, U5PWR.VDD, U5PWR.VDDA, U8.VCC, U8.WP
- net +5V: now also IC5.VI, LED4.A, PCB1.5V0@1, PCB1.5V0@2, Q1.S, SV2.3; no longer IC1.VI, JP5.5V0@1, JP5.5V0@2, Q2.S, SV1.3
- net +5V_RAW: now also $3_0_$_2018-08-14_21-12-08.VOUT+; no longer PCB1.VOUT+
- net +7V/1: now also JP3.2, LED2.A, SV2.1; no longer JP4.2, SV1.1
- net +7V/2: now also JP1.2, LED3.A, SV2.2; no longer JP3.2, SV1.2
- net 3V3_RPI: now also PCB1.3V3@1; no longer JP5.3V3@1
- net 3V3_STABILIZED: now also IC5.VO; no longer IC1.VO
- net 5V_NOT_TRIMMED: now also Q1.D; no longer Q2.D
- net BAT_MEAS: now also R7.1, R8.2, U1PA.PA4; no longer R11.1, R12.2, U5PA.PA4
- net BOOT0: now also R5.2, U1CTL.BOOT0; no longer R9.2, U5CTL.BOOT0
- net D1-R3: now also Q1.G, R6.2; no longer Q2.G, R10.2
- net DATA_N: now also J1.D-; no longer J2.D-
- net DATA_P: now also J1.D+; no longer J2.D+
- net EN1: now also IC1.PWM, U1PA.PA6; no longer U1.PWM, U5PA.PA6
- net EN2: now also U1PA.PA7; no longer U5PA.PA7
- net EN3: now also IC2.PWM, U1PB.PB0; no longer U2.PWM, U5PB.PB0
- net EN4: now also U1PB.PB1; no longer U5PB.PB1
- net GND: now also $3_0_$_2018-08-14_21-12-08.VIN-, $3_0_$_2018-08-14_21-12-08.VOUT-, IC1.DIS, IC1.GND@1, IC1.GND@2, IC2.DIS, IC2.GND@1, IC2.GND@2, IC5.GND, J1.GND, J1.SHEILD, JP1.3, PCB1.GND@1, PCB1.GND@2, PCB1.GND@3, PCB1.GND@4, PCB1.GND@5, PCB1.GND@6, PCB1.GND@7, PCB1.GND@8, R10.2, R11.2, R12.2, R13.2, R5.1, R6.1, R8.1, R9.2, SV1.3, SV2.10, SV2.9, U1PWR.VSS, U1PWR.VSSA, U2.A1, U2.A2, U2.VSS; no longer IC1.GND, J2.GND, J2.SHEILD, JP10.3, JP4.3, JP5.GND@1, JP5.GND@2, JP5.GND@3, JP5.GND@4, JP5.GND@5, JP5.GND@6, JP5.GND@7, JP5.GND@8, PCB1.VIN-, PCB1.VOUT-, R10.1, R12.1, R9.1, SV1.10, SV1.9, U1.DIS, U1.GND@1, U1.GND@2, U2.DIS, U2.GND@1, U2.GND@2, U5PWR.VSS, U5PWR.VSSA, U8.A1, U8.A2, U8.VSS
- net IN11: now also IC1.DIR, U1PB.PB8; no longer U1.DIR, U5PB.PB8
- net IN21: now also U1PA.PA11; no longer U5PA.PA11
- net IN31: now also IC2.DIR, U1PB.PB12; no longer U2.DIR, U5PB.PB12
- net IN41: now also U1PB.PB14; no longer U5PB.PB14
- net LED: now also U1PA.PA5; no longer U5PA.PA5
- net MOT11: now also IC1.OUT1; no longer U1.OUT1
- net MOT12: now also IC1.OUT2; no longer U1.OUT2
- net MOT31: now also IC2.OUT1; no longer U2.OUT1
- net MOT32: now also IC2.OUT2; no longer U2.OUT2
- net N$14: now also Q2B.S2, RN1C.1; no longer Q4B.S2, RN2C.1
- net N$16: now also Q2B.D2, RN1D.1; no longer Q4B.D2, RN2D.1
- net N$8: now also SV1.6; no longer JP10.6
- net NRST: now also PCB1.GPIO18, R4.1, SV1.5, U1CTL.NRST; no longer JP10.5, JP5.GPIO18, R8.1, U5CTL.NRST
- net OSCILATOR_N: now also U1CTL.PF0-OSC_IN, Y1.2; no longer Q1.2, U5CTL.PF0-OSC_IN
- net OSCILATOR_P: now also U1CTL.PF1-OSC_OUT, Y1.1; no longer Q1.1, U5CTL.PF1-OSC_OUT
- net RPI_CLK: now also IC1.SCK, IC2.SCK, PCB1.GPIO11/SCLK, U1PB.PB3; no longer JP5.GPIO11/SCLK, U1.SCK, U2.SCK, U5PB.PB3
- net RPI_MISO: now also PCB1.GPIO09/MISO, U1PB.PB4; no longer JP5.GPIO09/MISO, U5PB.PB4
- net RPI_MOSI: now also IC1.SI, PCB1.GPIO10/MOSI, U1PB.PB5; no longer JP5.GPIO10/MOSI, U1.SI, U5PB.PB5
- net RPI_RXD: now also PCB1.RXD0/GPIO15, U1PB.PB6; no longer JP5.RXD0/GPIO15, U5PB.PB6
- net RPI_TXD: now also PCB1.TXD0/GPIO14, U1PB.PB7; no longer JP5.TXD0/GPIO14, U5PB.PB7
- net SCL: now also PCB1.GPIO03/SCL1, R3.1, U1PA.PF6, U2.SCL; no longer JP5.GPIO03/SCL1, R7.1, U5PA.PF6, U8.SCL
- net SCL_TX: now also SV2.5, U1PB.PB10; no longer SV1.5, U5PB.PB10
- net SDA: now also PCB1.GPIO02/SDA1, R2.1, U1PA.PF7, U2.SDA; no longer JP5.GPIO02/SDA1, R6.1, U5PA.PF7, U8.SDA
- net SDA_RX: now also SV2.4, U1PB.PB11; no longer SV1.4, U5PB.PB11
- net SEN1: now also U1PA.PA0; no longer U5PA.PA0
- net SEN2: now also U1PA.PA1; no longer U5PA.PA1
- net SEN3: now also U1PA.PA2; no longer U5PA.PA2
- net SEN4: now also U1PA.PA3; no longer U5PA.PA3
- net SERVO1: now also JP1.1, RN2D.1, SV2.6; no longer JP2.1, RN1D.1, SV1.6
- net SERVO1_UC: now also RN2C.1, U1PA.PA8; no longer RN1C.1, U5PA.PA8
- net SERVO2: now also JP2.1, RN2B.1, SV2.7; no longer JP3.1, RN1B.1, SV1.7
- net SERVO2_UC: now also RN2A.1, U1PA.PA9; no longer RN1A.1, U5PA.PA9
- net SERVO3: now also JP3.1, Q2A.D1, RN1B.1, SV2.8; no longer JP4.1, Q4A.D1, RN2B.1, SV1.8
- net SERVO3_UC: now also Q2A.S1, RN1A.1, U1PA.PA10; no longer Q4A.S1, RN2A.1, U5PA.PA10
- net SO1-SI3: now also IC1.SO; no longer U1.SO
- net SO2-SI4: now also IC2.SO; no longer U2.SO
- net SO3-SI2: now also IC2.SI; no longer U2.SI
- net SPI1_NSS: now also PCB1.!CE0!/GPIO08, R1.1, U1PA.PA15; no longer JP5.!CE0!/GPIO08, R5.1, U5PA.PA15
- net SWCLK: now also PCB1.GEN6/GPIO25, SV1.1, U1PA.PA14-SWCLK; no longer JP10.1, JP5.GEN6/GPIO25, U5PA.PA14-SWCLK
- net SWDIO: now also PCB1.GEN5/GPIO24, SV1.2, U1PA.PA13-SWDIO; no longer JP10.2, JP5.GEN5/GPIO24, U5PA.PA13-SWDIO
- net TLE_NSS: now also IC1.CS_N, IC2.CS_N, U1PB.PB2; no longer U1.CS_N, U2.CS_N, U5PB.PB2
- net VCC: now also $3_0_$_2018-08-14_21-12-08.VIN+, IC1.VS, IC2.VS, LED1.A, R7.2; no longer PCB1.VIN+, R11.2, U1.VS, U2.VS

Commit message: change few footprints, complete wiring
Parts:
- RN1, RN2: value (none) -> 1k; device electronics-shield:RESISTOR-DIL_4R-NEXB38V -> SparkFun-Resistors:1KOHM-ARRAY(4)-0805_ARV-1/10W-5%
Connections:
- net N$14: now also RN2C.1; no longer RN1C.1
- net N$16: now also RN2D.1; no longer RN1D.1
- net SERVO1: now also RN1D.1; no longer RN2D.1
- net SERVO1_UC: now also RN1C.1; no longer RN2C.1
- net SERVO2: now also RN1B.1; no longer RN2B.1
- net SERVO2_UC: now also RN1A.1; no longer RN2A.1
- net SERVO3: now also RN2B.1; no longer RN1B.1
- net SERVO3_UC: now also RN2A.1; no longer RN1A.1
Changed lines of the file:
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@@
 <?xml version="1.0" encoding="utf-8"?>
 <!DOCTYPE eagle SYSTEM "eagle.dtd">
-<eagle version="9.1.2">
+<eagle version="9.1.3">
 <drawing>
 <settings>
@@
 <part name="GND36" library="electronics-shield" deviceset="SUPPLY1_GND*?:1" device=""/>
 <part name="P+3" library="electronics-shield" deviceset="SUPPLY1_+5V" device=""/>
-<part name="X2" library="Kell Ideas" library_urn="urn:adsk.eagle:library:4431361" deviceset="CONNECTOR_PHOENIX" device="" package3d_urn="urn:adsk.eagle:package:4691404/3" value="Listwa zaciskowa rozłączalna 3.50mm 8pin kątowe 90° gniazdo"/>
+<part name="X2" library="Kell Ideas" library_urn="urn:adsk.eagle:library:4431361" deviceset="CONNECTOR_PHOENIX" device="" package3d_urn="urn:adsk.eagle:package:4691404/4" value="Listwa zaciskowa rozłączalna 3.50mm 8pin kątowe 90° gniazdo"/>
 <part name="SUPPLY13" library="electronics-shield" deviceset="SUPPLY2_+7V" device="" value="+7V/1"/>
 <part name="SUPPLY14" library="electronics-shield" deviceset="SUPPLY2_+7V" device="" value="+7V/2"/>
@@
 <part name="IC5" library="electronics-shield" deviceset="LINEAR_MCP1703" device="CB"/>
 <part name="Q3" library="electronics-shield" deviceset="ON-SEMICONDUCTOR---NTZD3154NT1G_ON_SEMICONDUCTOR_NTZD3154NT1G" device="ON_SEMICONDUCTOR_NTZD3154NT1G_0_0"/>
-<part name="RN2" library="electronics-shield" deviceset="RESISTOR-DIL_4R-N" device="EXB38V"/>
 <part name="Q2" library="electronics-shield" deviceset="ON-SEMICONDUCTOR---NTZD3154NT1G_ON_SEMICONDUCTOR_NTZD3154NT1G" device="ON_SEMICONDUCTOR_NTZD3154NT1G_0_0"/>
-<part name="RN1" library="electronics-shield" deviceset="RESISTOR-DIL_4R-N" device="EXB38V"/>
 <part name="SJ1" library="Kell Ideas" library_urn="urn:adsk.eagle:library:4431361" deviceset="SOLDER_JUMPER" device="" package3d_urn="urn:adsk.eagle:package:4689481/4"/>
 <part name="SJ2" library="Kell Ideas" library_urn="urn:adsk.eagle:library:4431361" deviceset="SOLDER_JUMPER" device="" package3d_urn="urn:adsk.eagle:package:4689481/4"/>
@@
 <part name="P+6" library="supply1" library_urn="urn:adsk.eagle:library:371" deviceset="VCC" device=""/>
 <part name="GND44" library="supply1" library_urn="urn:adsk.eagle:library:371" deviceset="GND" device=""/>
+<part name="RN1" library="SparkFun-Resistors" library_urn="urn:adsk.eagle:library:532" deviceset="1KOHM-ARRAY(4)" device="-0805_ARV-1/10W-5%" package3d_urn="urn:adsk.eagle:package:39659/1" value="1k"/>
+<part name="RN2" library="SparkFun-Resistors" library_urn="urn:adsk.eagle:library:532" deviceset="1KOHM-ARRAY(4)" device="-0805_ARV-1/10W-5%" package3d_urn="urn:adsk.eagle:package:39659/1" value="1k"/>
 </parts>
 <sheets>
@@
 <instance part="Q3" gate="A" x="60.96" y="132.08" rot="R270"/>
 <instance part="Q3" gate="B" x="134.62" y="132.08" rot="R270"/>
-<instance part="RN2" gate="A" x="40.64" y="134.62" rot="R90"/>
-<instance part="RN2" gate="B" x="63.5" y="134.62" rot="R90"/>
-<instance part="RN2" gate="C" x="114.3" y="134.62" rot="R90"/>
-<instance part="RN2" gate="D" x="139.7" y="134.62" rot="R90"/>
 <instance part="Q2" gate="A" x="58.42" y="78.74" rot="R270"/>
 <instance part="Q2" gate="B" x="132.08" y="78.74" rot="R270"/>
-<instance part="RN1" gate="A" x="38.1" y="81.28" rot="R90"/>
-<instance part="RN1" gate="B" x="60.96" y="81.28" rot="R90"/>
-<instance part="RN1" gate="C" x="111.76" y="81.28" rot="R90"/>
-<instance part="RN1" gate="D" x="137.16" y="81.28" rot="R90"/>
+<instance part="RN1" gate="B" x="63.5" y="134.62" rot="R90"/>
+<instance part="RN1" gate="C" x="114.3" y="134.62" rot="R90"/>
+<instance part="RN1" gate="D" x="139.7" y="134.62" rot="R90"/>
+<instance part="RN1" gate="A" x="40.64" y="134.62" rot="R90"/>
+<instance part="RN2" gate="B" x="60.96" y="81.28" rot="R90"/>
+<instance part="RN2" gate="C" x="111.76" y="81.28" rot="R90"/>
+<instance part="RN2" gate="D" x="137.16" y="81.28" rot="R90"/>
+<instance part="RN2" gate="A" x="38.1" y="81.28" rot="R90"/>
 </instances>
 <busses>
@@
 <net name="+3V3" class="3">
 <segment>
-<pinref part="RN2" gate="A" pin="2"/>
 <wire x1="40.64" y1="139.7" x2="40.64" y2="142.24" width="0.1524" layer="91"/>
 <wire x1="40.64" y1="142.24" x2="53.34" y2="142.24" width="0.1524" layer="91"/>
@@
 <junction x="40.64" y="142.24"/>
 <label x="40.64" y="152.4" size="1.778" layer="95" rot="R90"/>
-</segment>
-<segment>
 <pinref part="RN1" gate="A" pin="2"/>
+</segment>
+<segment>
 <wire x1="38.1" y1="86.36" x2="38.1" y2="88.9" width="0.1524" layer="91"/>
 <wire x1="38.1" y1="88.9" x2="50.8" y2="88.9" width="0.1524" layer="91"/>
@@
 <junction x="38.1" y="88.9"/>
 <label x="38.1" y="99.06" size="1.778" layer="95"/>
-</segment>
-<segment>
-<pinref part="RN2" gate="C" pin="2"/>
+<pinref part="RN2" gate="A" pin="2"/>
+</segment>
+<segment>
 <wire x1="114.3" y1="139.7" x2="114.3" y2="142.24" width="0.1524" layer="91"/>
 <pinref part="Q3" gate="B" pin="G2"/>
@@
 <junction x="114.3" y="142.24"/>
 <label x="114.3" y="152.4" size="1.778" layer="95"/>
-</segment>
-<segment>
 <pinref part="RN1" gate="C" pin="2"/>
+</segment>
+<segment>
 <wire x1="111.76" y1="86.36" x2="111.76" y2="88.9" width="0.1524" layer="91"/>
 <pinref part="Q2" gate="B" pin="G2"/>
@@
 <junction x="111.76" y="88.9"/>
 <label x="111.76" y="99.06" size="1.778" layer="95"/>
+<pinref part="RN2" gate="C" pin="2"/>
 </segment>
 </net>
 <net name="+5V" class="3">
 <segment>
-<pinref part="RN2" gate="B" pin="2"/>
 <wire x1="63.5" y1="139.7" x2="63.5" y2="152.4" width="0.1524" layer="91"/>
 <label x="63.5" y="154.94" size="1.778" layer="95" rot="R90"/>
-</segment>
-<segment>
 <pinref part="RN1" gate="B" pin="2"/>
+</segment>
+<segment>
 <wire x1="60.96" y1="86.36" x2="60.96" y2="99.06" width="0.1524" layer="91"/>
 <label x="60.96" y="99.06" size="1.778" layer="95"/>
-</segment>
-<segment>
-<pinref part="RN2" gate="D" pin="2"/>
+<pinref part="RN2" gate="B" pin="2"/>
+</segment>
+<segment>
 <wire x1="139.7" y1="139.7" x2="139.7" y2="152.4" width="0.1524" layer="91"/>
 <label x="139.7" y="152.4" size="1.778" layer="95"/>
-</segment>
-<segment>
 <pinref part="RN1" gate="D" pin="2"/>
+</segment>
+<segment>
 <wire x1="137.16" y1="86.36" x2="137.16" y2="99.06" width="0.1524" layer="91"/>
 <label x="137.16" y="99.06" size="1.778" layer="95"/>
+<pinref part="RN2" gate="D" pin="2"/>
 </segment>
 </net>
@@
 <pinref part="Q3" gate="A" pin="S1"/>
 <wire x1="45.72" y1="124.46" x2="40.64" y2="124.46" width="0.1524" layer="91"/>
-<pinref part="RN2" gate="A" pin="1"/>
 <wire x1="40.64" y1="124.46" x2="25.4" y2="124.46" width="0.1524" layer="91"/>
 <wire x1="40.64" y1="129.54" x2="40.64" y2="124.46" width="0.1524" layer="91"/>
 <junction x="40.64" y="124.46"/>
 <label x="20.32" y="124.46" size="1.778" layer="95"/>
+<pinref part="RN1" gate="A" pin="1"/>
 </segment>
 </net>
 <net name="SERVO2" class="0">
 <segment>
-<pinref part="RN2" gate="B" pin="1"/>
 <pinref part="Q3" gate="A" pin="D1"/>
 <wire x1="63.5" y1="129.54" x2="63.5" y2="124.46" width="0.1524" layer="91"/>
@@
 <junction x="63.5" y="124.46"/>
 <label x="66.04" y="124.46" size="1.778" layer="95"/>
+<pinref part="RN1" gate="B" pin="1"/>
 </segment>
 </net>
 <net name="SERVO3" class="0">
 <segment>
-<pinref part="RN1" gate="B" pin="1"/>
 <pinref part="Q2" gate="A" pin="D1"/>
 <wire x1="60.96" y1="76.2" x2="60.96" y2="71.12" width="0.1524" layer="91"/>
@@
 <junction x="60.96" y="71.12"/>
 <label x="63.5" y="71.12" size="1.778" layer="95"/>
+<pinref part="RN2" gate="B" pin="1"/>
 </segment>
 </net>
@@
 <segment>
 <pinref part="Q2" gate="B" pin="S2"/>
-<pinref part="RN1" gate="C" pin="1"/>
 <wire x1="116.84" y1="71.12" x2="111.76" y2="71.12" width="0.1524" layer="91"/>
 <wire x1="111.76" y1="71.12" x2="111.76" y2="76.2" width="0.1524" layer="91"/>
 <wire x1="111.76" y1="71.12" x2="104.14" y2="71.12" width="0.1524" layer="91"/>
 <junction x="111.76" y="71.12"/>
+<pinref part="RN2" gate="C" pin="1"/>
 </segment>
 </net>
 <net name="N$16" class="0">
 <segment>
-<pinref part="RN1" gate="D" pin="1"/>
 <pinref part="Q2" gate="B" pin="D2"/>
 <wire x1="137.16" y1="76.2" x2="137.16" y2="71.12" width="0.1524" layer="91"/>
@@
 <wire x1="137.16" y1="71.12" x2="142.24" y2="71.12" width="0.1524" layer="91"/>
 <junction x="137.16" y="71.12"/>
+<pinref part="RN2" gate="D" pin="1"/>
 </segment>
 </net>
@@
 <pinref part="Q2" gate="A" pin="S1"/>
 <wire x1="43.18" y1="71.12" x2="38.1" y2="71.12" width="0.1524" layer="91"/>
-<pinref part="RN1" gate="A" pin="1"/>
 <wire x1="38.1" y1="71.12" x2="22.86" y2="71.12" width="0.1524" layer="91"/>
 <wire x1="38.1" y1="76.2" x2="38.1" y2="71.12" width="0.1524" layer="91"/>
 <junction x="38.1" y="71.12"/>
 <label x="20.32" y="71.12" size="1.778" layer="95"/>
+<pinref part="RN2" gate="A" pin="1"/>
 </segment>
 </net>
@@
 <segment>
 <pinref part="Q3" gate="B" pin="S2"/>
-<pinref part="RN2" gate="C" pin="1"/>
 <wire x1="119.38" y1="124.46" x2="114.3" y2="124.46" width="0.1524" layer="91"/>
 <wire x1="114.3" y1="124.46" x2="114.3" y2="129.54" width="0.1524" layer="91"/>
@@
 <junction x="114.3" y="124.46"/>
 <label x="96.52" y="124.46" size="1.778" layer="95"/>
+<pinref part="RN1" gate="C" pin="1"/>
 </segment>
 </net>
 <net name="SERVO1" class="0">
 <segment>
-<pinref part="RN2" gate="D" pin="1"/>
 <pinref part="Q3" gate="B" pin="D2"/>
 <wire x1="139.7" y1="129.54" x2="139.7" y2="124.46" width="0.1524" layer="91"/>
@@
 <junction x="139.7" y="124.46"/>
 <label x="142.24" y="124.46" size="1.778" layer="95"/>
-</segment>
-</net>
+<pinref part="RN1" gate="D" pin="1"/>
+</segment>
+</net>

Commit message: Changed microprocessor, major and minor changes
Parts:
- removed $3_0_$_2018-08-14_21-12-08, $3_1_$_2018-08-14_21-12-08, $3_2_$_2018-08-14_21-12-08: Moduł przetwornicy DC-DC Step-down 4.5..28V --- regulowane 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, Kell Ideas:MP1584_MODULE
- removed C10: 1u, Kell Ideas:CAPACITOR_SMD
- removed C11, C12, C13, C14, C6, C9: 100n, Kell Ideas:CAPACITOR_SMD
- removed C15: 4.7uF, Kell Ideas:CAPACITOR_SMD
- removed C16: 1uF, Kell Ideas:CAPACITOR_SMD
- removed C17: 100u, Kell Ideas:CAPACITOR_POL_SMD
- removed C18: 22u, Kell Ideas:CAPACITOR_SMD
- removed C5: 4u7, Kell Ideas:CAPACITOR_SMD
- removed C7, C8: 20p, Kell Ideas:CAPACITOR_SMD
- removed D17: SMBJ5.0A-TR, Kell Ideas:SUPPRESSOR-SMBJ
- removed F1, F2, F3: SL125-33, Kell Ideas:PPTCD
- removed IC5: LINEAR_MCP1703CB, electronics-shield:LINEAR_MCP1703CB
- removed Q1: USER-SUBMITTED_MOSFET-PCHANNELSMD, electronics-shield:USER-SUBMITTED_MOSFET-PCHANNELSMD
- removed R1, R4, R5, R7: 10k, Kell Ideas:RESISTOR_SMD
- removed R2, R3: 4k7, Kell Ideas:RESISTOR_SMD
- removed R6: 100k, Kell Ideas:RESISTOR_SMD
- removed R8: 1k, Kell Ideas:RESISTOR_SMD
- removed SJ1, SJ2: (no value), Kell Ideas:SOLDER_JUMPER
- removed U1: STM32F0XX8T, Kell Ideas:STM32F0XX8T
- removed Y1: 8 MHz, Kell Ideas:CRYSTAL
- added C35, C36, C37, C38, C39: ?, Kell Ideas:CAPACITOR_SMD_0402
- added C40, C41: (no value), rcl:CPOL-EU153CLV-0405
- added D20: 28V-5A, Seeed-Diode:SMD-DIODE-SCHOTTKY-28V-5A(DO-214AA)
- added IC6, IC7, IC8, IC9: ACS712-LC, allegro-2:ACS712-LC
- added L3: ?, SparkFun-Coils:INDUCTOR-CR54-47UH
- added R22, R23, R24, R25: ?, Kell Ideas:RESISTOR_SMD_0402
- added U5: AOZ1284, Kell Ideas:AOZ1284
- added U6: STM32F103VCT6, Kell Ideas:STM32F103VCT6
- C1, C19, C2, C20, C3, C4: device Kell Ideas:CAPACITOR_SMD -> Kell Ideas:CAPACITOR_SMD_0402
- R10, R11, R12, R13, R9: device Kell Ideas:RESISTOR_SMD -> Kell Ideas:RESISTOR_SMD_0402
Connections:
- removed net +5V_RAW: $3_0_$_2018-08-14_21-12-08.VOUT+, F1.2
- removed net +7V/1_RAW: $3_1_$_2018-08-14_21-12-08.VOUT+, F2.2
- removed net +7V/2_RAW: $3_2_$_2018-08-14_21-12-08.VOUT+, F3.1
- removed net 3V3_STABILIZED: C16.1, IC5.VO, SJ1.2
- removed net 5V_NOT_TRIMMED: C12.1, F1.1, Q1.D
- removed net BAT_MEAS: C18.1, R7.1, R8.2, U1PA.PA4
- removed net D1-R3: D17.A, Q1.G, R6.2
- removed net LED: U1PA.PA5
- removed net OSCILATOR_N: C7.2, U1CTL.PF0-OSC_IN, Y1.2
- removed net OSCILATOR_P: C8.2, U1CTL.PF1-OSC_OUT, Y1.1
- removed net SEN1: U1PA.PA0
- removed net SEN2: U1PA.PA1
- removed net SEN3: U1PA.PA2
- removed net SEN4: U1PA.PA3
- new net BS2: C38.1, U5.BST
- new net COMP: C37.1, U5.COMP
- new net C_COMP_R_COMP: C37.2, R25.2
- new net FB: R23.1, R24.2, U5.FB
- new net FSW1: R22.2, U5.FSW
- new net LX: C38.2, D20.-, L3.1, U5.LX
- new net N$10: U6B.VDDA, U6B.VDD_1, U6B.VDD_2, U6B.VDD_3, U6B.VDD_4, U6B.VDD_5
- new net N$7: IC1.VS, IC6.IP+, IC6.IP+1
- new net N$9: U6B.VREF-, U6B.VSSA, U6B.VSS_1, U6B.VSS_2, U6B.VSS_3, U6B.VSS_4, U6B.VSS_5
- new net NC: U6A.NC
- new net OSC_IN: U6A.OSC_IN
- new net OSC_OUT: U6A.OSC_OUT
- new net PA0-WKUP: U6A.PA0-WKUP
- new net PA1: U6A.PA1
- new net PA10: U6A.PA10
- new net PA11: U6A.PA11
- new net PA12: U6A.PA12
- new net PA13: U6A.PA13
- new net PA14: U6A.PA14
- new net PA15: U6A.PA15
- new net PA2: U6A.PA2
- new net PA3: U6A.PA3
- new net PA4: U6A.PA4
- new net PA5: U6A.PA5
- new net PA6: U6A.PA6
- new net PA7: U6A.PA7
- new net PA8: U6A.PA8
- new net PA9: U6A.PA9
- new net PB0: U6A.PB0
- new net PB1: U6A.PB1
- new net PB10: U6A.PB10
- new net PB11: U6A.PB11
- new net PB12: U6A.PB12
- new net PB13: U6A.PB13
- new net PB14: U6A.PB14
- new net PB15: U6A.PB15
- new net PB2: U6A.PB2
- new net PB3: U6A.PB3
- new net PB4: U6A.PB4
- new net PB5: U6A.PB5
- new net PB6: U6A.PB6
- new net PB7: U6A.PB7
- new net PB8: U6A.PB8
- new net PB9: U6A.PB9
- new net PC0: U6A.PC0
- new net PC1: U6A.PC1
- new net PC10: U6A.PC10
- new net PC11: U6A.PC11
- new net PC12: U6A.PC12
- new net PC13-TAMPER-RTC: U6A.PC13-TAMPER-RTC
- new net PC14-OSC32_IN: U6A.PC14-OSC32_IN
- new net PC15-OSC32_OUT: U6A.PC15-OSC32_OUT
- new net PC2: U6A.PC2
- new net PC3: U6A.PC3
- new net PC4: U6A.PC4
- new net PC5: U6A.PC5
- new net PC6: U6A.PC6
- new net PC7: U6A.PC7
- new net PC8: U6A.PC8
- new net PC9: U6A.PC9
- new net PD0: U6A.PD0
- new net PD1: U6A.PD1
- new net PD10: U6A.PD10
- new net PD11: U6A.PD11
- new net PD12: U6A.PD12
- new net PD13: U6A.PD13
- new net PD14: U6A.PD14
- new net PD15: U6A.PD15
- new net PD2: U6A.PD2
- new net PD3: U6A.PD3
- new net PD4: U6A.PD4
- new net PD5: U6A.PD5
- new net PD6: U6A.PD6
- new net PD7: U6A.PD7
- new net PD8: U6A.PD8
- new net PD9: U6A.PD9
- new net PE0: U6A.PE0
- new net PE1: U6A.PE1
- new net PE10: U6A.PE10
- new net PE11: U6A.PE11
- new net PE12: U6A.PE12
- new net PE13: U6A.PE13
- new net PE14: U6A.PE14
- new net PE15: U6A.PE15
- new net PE2: U6A.PE2
- new net PE3: U6A.PE3
- new net PE4: U6A.PE4
- new net PE5: U6A.PE5
- new net PE6: U6A.PE6
- new net PE7: U6A.PE7
- new net PE8: U6A.PE8
- new net PE9: U6A.PE9
- new net SS1: C39.2, U5.SS
- net +3V3: no longer C10.1, C11.1, C5.1, C6.1, C9.1, R1.2, R2.2, R3.2, R4.2, SJ1.1, SJ2.1, U1PWR.VDD, U1PWR.VDDA
- net +5V: now also C35.1, C40.+, L3.2, R23.2; no longer C15.1, D17.C, IC5.VI, Q1.S
- net +7V/1: no longer C13.1, F2.1
- net +7V/2: no longer C14.1, F3.2
- net 3V3_RPI: no longer SJ2.2
- net BOOT0: now also U6A.BOOT0; no longer R5.2, U1CTL.BOOT0
- net EN1: no longer U1PA.PA6
- net EN2: no longer U1PA.PA7
- net EN3: no longer U1PB.PB0
- net EN4: no longer U1PB.PB1
- net GND: now also C35.2, C36.2, C39.1, C40.-, C41.-, D20.+, R22.1, R24.1, R25.1, U5.GND; no longer $3_0_$_2018-08-14_21-12-08.VIN-, $3_0_$_2018-08-14_21-12-08.VOUT-, $3_1_$_2018-08-14_21-12-08.VIN-, $3_1_$_2018-08-14_21-12-08.VOUT-, $3_2_$_2018-08-14_21-12-08.VIN-, $3_2_$_2018-08-14_21-12-08.VOUT-, C10.2, C11.2, C12.2, C13.2, C14.2, C15.2, C16.2, C17.-, C18.2, C5.2, C6.2, C7.1, C8.1, C9.2, IC5.GND, R5.1, R6.1, R8.1, U1PWR.VSS, U1PWR.VSSA
- net IN11: no longer U1PB.PB8
- net IN21: no longer U1PA.PA11
- net IN31: no longer U1PB.PB12
- net IN41: no longer U1PB.PB14
- net MOT11: now also X2-8.K; no longer X2-7.K
- net MOT12: now also X2-7.K; no longer X2-8.K
- net MOT21: now also X2-6.K; no longer X2-5.K
- net MOT22: now also X2-5.K; no longer X2-6.K
- net MOT31: now also X2-4.K; no longer X2-3.K
- net MOT32: now also X2-3.K; no longer X2-4.K
- net MOT41: now also X2-2.K; no longer X2-1.K
- net MOT42: now also X2-1.K; no longer X2-2.K
- net NRST: now also U6A.NRST; no longer R4.1, U1CTL.NRST
- net RPI_CLK: no longer U1PB.PB3
- net RPI_MISO: no longer U1PB.PB4
- net RPI_MOSI: no longer U1PB.PB5
- net RPI_RXD: no longer U1PB.PB6
- net RPI_TXD: no longer U1PB.PB7
- net SCL: no longer R3.1, U1PA.PF6
- net SCL_TX: no longer U1PB.PB10
- net SDA: no longer R2.1, U1PA.PF7
- net SDA_RX: no longer U1PB.PB11
- net SERVO1_UC: no longer U1PA.PA8
- net SERVO2_UC: no longer U1PA.PA9
- net SERVO3_UC: no longer U1PA.PA10
- net SPI1_NSS: no longer R1.1, U1PA.PA15
- net SWCLK: no longer U1PA.PA14-SWCLK
- net SWDIO: no longer U1PA.PA13-SWDIO
- net TLE_NSS: no longer U1PB.PB2
- net VCC: now also C36.1, C41.+, IC6.IP-, IC6.IP-1, U5.VIN_PAD; no longer $3_0_$_2018-08-14_21-12-08.VIN+, $3_1_$_2018-08-14_21-12-08.VIN+, $3_2_$_2018-08-14_21-12-08.VIN+, C17.+, IC1.VS, R7.2
Other:
- note removed: "Battery Measurement"
- note removed: "I2C2"
- note removed: "Power Supply Raspberry 5V / 3A"
- note removed: "Power Supply Servo 7V / 3 A"
- note removed: "Second Servo PS 7V / 3 A"
